File: board_8x8_stm32/8x8_stm32.sch (EAGLE design)
At the start: 121 parts, among them IC1 STM32F0, J1 SWD_SHROUD, Q1 BSS123, Q10 BSS84, Q11 BSS84, Q12 BSS84, Q13 BSS84, Q14 BSS84, Q15 BSS84, Q16 BSS84, Q2 BSS123, Q3 BSS123, Q4 BSS123, Q5 BSS123, Q6 BSS123, Q7 BSS123, Q8 BSS123, Q9 BSS84

Commit message: almost done
Parts:
- added J2: (no value), tag-connect:TC2030-MCP-NL
- added T1: (no value), transistor-neu-to92:-NPN-TO92
- added T2: (no value), transistor-neu-to92:-NPN-TO92-BCE
Connections:
- new net N$12: J2.VDD
- new net N$13: J2.VSS(GND)
- new net N$14: J2.ICSP_DAT/PGD
- new net N$15: J2.ICSP_CLK/PGC
Changed lines of the file:
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@@
 <part name="SJ2" library="SparkFun-Passives" deviceset="JUMPER-PAD-2-NC_BY_TRACE" device="" value=""/>
 <part name="C16" library="passives-7351" deviceset="CAPACITOR" device="0603-N"/>
+<part name="T1" library="transistor-neu-to92" deviceset="*-NPN-" device="TO92"/>
+<part name="T2" library="transistor-neu-to92" deviceset="*-NPN-" device="TO92-BCE"/>
+<part name="J2" library="tag-connect" deviceset="TC2030" device="-MCP-NL"/>
 </parts>
 <sheets>
@@
 <instance part="SJ2" gate="G$1" x="91.44" y="83.82"/>
 <instance part="C16" gate="G$1" x="-15.24" y="68.58"/>
+<instance part="T1" gate="G$1" x="91.44" y="-25.4"/>
+<instance part="T2" gate="G$1" x="99.06" y="-17.78"/>
+<instance part="J2" gate="G$1" x="43.18" y="162.56"/>
 </instances>
 <busses>
@@
 </segment>
 </net>
+<net name="N$12" class="0">
+<segment>
+<pinref part="J2" gate="G$1" pin="VDD"/>
+<wire x1="30.48" y1="167.64" x2="22.86" y2="167.64" width="0.1524" layer="91"/>
+</segment>
+</net>
+<net name="N$13" class="0">
+<segment>
+<pinref part="J2" gate="G$1" pin="VSS(GND)"/>
+<wire x1="22.86" y1="165.1" x2="30.48" y2="165.1" width="0.1524" layer="91"/>
+</segment>
+</net>
+<net name="N$14" class="0">
+<segment>
+<pinref part="J2" gate="G$1" pin="ICSP_DAT/PGD"/>
+<wire x1="30.48" y1="162.56" x2="22.86" y2="162.56" width="0.1524" layer="91"/>
+</segment>
+</net>
+<net name="N$15" class="0">
+<segment>
+<pinref part="J2" gate="G$1" pin="ICSP_CLK/PGC"/>
+<wire x1="22.86" y1="160.02" x2="30.48" y2="160.02" width="0.1524" layer="91"/>
+</segment>
+</net>
