File: board_8x8_stm32/8x8_stm32.sch (EAGLE design)
At the start: 124 parts, among them IC1 STM32F0, J1 SWD_SHROUD, Q1 BSS123, Q10 BSS84, Q11 BSS84, Q12 BSS84, Q13 BSS84, Q14 BSS84, Q15 BSS84, Q16 BSS84, Q2 BSS123, Q3 BSS123, Q4 BSS123, Q5 BSS123, Q6 BSS123, Q7 BSS123, Q8 BSS123, Q9 BSS84

Commit message: first prototype almost done
Parts:
- removed J2: (no value), tag-connect:TC2030-MCP-NL
- removed RN1, RN2: (no value), resistor-dil:4R-NEXB38V
- removed T1: (no value), transistor-neu-to92:-NPN-TO92
- removed T2: (no value), transistor-neu-to92:-NPN-TO92-BCE
- added JP7: TC2030-SWDNL, tag-connect:TC2030-SWDNL
- added R11, R12, R13, R14, R15, R16, R17, R18: (no value), passives-7351:RESISTOR0603-N
- C1: value 100p -> (none); device passives-7351:CAPACITOR0603-N -> rcl:CPOL-EUE2-4
- C10, C9: value (none) -> 100p
- C12: device rcl:CPOL-EUE2-4 -> passives-7351:CAPACITOR0603-N
- C13: value (none) -> 100p; device rcl:CPOL-EUE2-4 -> passives-7351:CAPACITOR0603-N
- C14, C15: value (none) -> 100p; device rcl:C-EU050-025X075 -> passives-7351:CAPACITOR0603-N
- C16: device passives-7351:CAPACITOR0603-N -> rcl:CPOL-EUE2-4
- C2, C3: value 100p -> (none); device passives-7351:CAPACITOR0603-N -> rcl:C-EU050-025X075
- C5, C6: value 100p -> (none)
- JP1: device Mine:M02PTH -> SparkFun-Connectors:M08
- JP2: device SparkFun-Connectors:M06SILK_FEMALE_PTH -> SparkFun-Connectors:M08
- JP5: device SparkFun-Connectors:M08 -> SparkFun-Connectors:M06SILK_FEMALE_PTH
- JP6: device SparkFun-Connectors:M08 -> Mine:M02PTH
- Q1, Q2, Q3: value BSS123 -> BSS84; device transistor-small-signal:BSS123 -> transistor-small-signal:BSS84
- Q10, Q11, Q9: value BSS84 -> BSS123; device transistor-small-signal:BSS84 -> transistor-small-signal:BSS123
- R10: value 2k2 -> (none)
- R2: value DNP -> 2k2
- R9: value (none) -> DNP
- renumbered U$1 to Q17
Connections:
- removed net N$1: Q8.D, RN2A.1
- removed net N$2: Q7.D, RN2B.1
- removed net N$3: Q6.D, RN2C.1
- removed net N$4: Q5.D, RN2D.1
- removed net N$5: Q4.D, RN1A.1
- removed net N$6: Q3.D, RN1B.1
- removed net N$7: Q2.D, RN1C.1
- removed net N$8: Q1.D, RN1D.1
- new net N$16: Q13.D, R15.P$2
- new net N$17: Q14.D, R16.P$2
- new net N$18: Q15.D, R17.P$2
- new net N$19: Q16.D, R18.P$2
- net +3V3: now also C12.1, C2.1, C5.1, C6.1, JP1.5, JP2.5, JP5.4, JP7.VCC, R10.P$2; no longer C10.1, C15.1, C16.1, C9.1, JP2.4, JP5.5, JP6.5, R9.P$2
- net +5V: now also C1.+, C16.+, C3.1, JP1.1, JP1.8, JP2.1, JP2.8, Q1.S, Q2.S, Q3.S; no longer C12.+, C13.+, C14.1, JP5.1, JP5.8, JP6.1, JP6.8, Q10.S, Q11.S, Q9.S
- net CFET1: now also Q11.G; no longer Q1.G
- net CFET2: now also Q10.G; no longer Q2.G
- net CFET3: now also Q9.G; no longer Q3.G
- net CFET4: now also Q8.G; no longer Q4.G
- net CFET5: now also Q7.G; no longer Q5.G
- net CFET7: now also Q5.G; no longer Q7.G
- net CFET8: now also Q4.G; no longer Q8.G
- net COL1: now also C14.1, LED16.C, LED24.C, LED32.C, LED40.C, LED48.C, LED56.C, LED64.C, LED8.C, Q4.D, R8.P$2; no longer C6.1, LED1.C, LED17.C, LED25.C, LED33.C, LED41.C, LED49.C, LED57.C, LED9.C, R6.P$2, RN2A.2
- net COL2: now also C13.1, LED15.C, LED23.C, LED31.C, LED39.C, LED47.C, LED55.C, LED63.C, LED7.C, Q5.D, R7.P$2; no longer C5.1, LED10.C, LED18.C, LED2.C, LED26.C, LED34.C, LED42.C, LED50.C, LED58.C, R5.P$2, RN2B.2
- net COL3: now also C7.1, LED14.C, LED22.C, LED30.C, LED38.C, LED46.C, LED54.C, LED6.C, LED62.C, Q6.D; no longer C3.1, LED11.C, LED19.C, LED27.C, LED3.C, LED35.C, LED43.C, LED51.C, LED59.C, RN2C.2
- net COL4: now also C9.1, LED13.C, LED21.C, LED29.C, LED37.C, LED45.C, LED5.C, LED53.C, LED61.C, Q7.D, R6.P$2; no longer C4.1, LED12.C, LED20.C, LED28.C, LED36.C, LED4.C, LED44.C, LED52.C, LED60.C, R4.P$2, RN2D.2
- net COL5: now also C15.1, LED12.C, LED20.C, LED28.C, LED36.C, LED4.C, LED44.C, LED52.C, LED60.C, Q8.D, R9.P$2; no longer C7.1, LED13.C, LED21.C, LED29.C, LED37.C, LED45.C, LED5.C, LED53.C, LED61.C, R7.P$2, RN1A.2
- net COL6: now also C8.1, LED11.C, LED19.C, LED27.C, LED3.C, LED35.C, LED43.C, LED51.C, LED59.C, Q9.D, R4.P$2; no longer C2.1, LED14.C, LED22.C, LED30.C, LED38.C, LED46.C, LED54.C, LED6.C, LED62.C, R2.P$2, RN1B.2
- net COL7: now also C10.1, LED10.C, LED18.C, LED2.C, LED26.C, LED34.C, LED42.C, LED50.C, LED58.C, Q10.D, R5.P$2; no longer C1.1, LED15.C, LED23.C, LED31.C, LED39.C, LED47.C, LED55.C, LED63.C, LED7.C, R1.P$2, RN1C.2
- net COL8: now also C4.1, LED1.C, LED17.C, LED25.C, LED33.C, LED41.C, LED49.C, LED57.C, LED9.C, Q11.D, R1.P$2, R2.P$1; no longer C8.1, LED16.C, LED24.C, LED32.C, LED40.C, LED48.C, LED56.C, LED64.C, LED8.C, R10.P$1, R8.P$2, RN1D.2
- net COMMS_DOWN: now also JP4.3; no longer JP5.3
- net COMMS_LEFT: now also JP2.3; no longer JP4.3
- net COMMS_UP: now also JP1.3; no longer JP6.3
- net GND: now also C1.-, C12.2, C13.2, C16.-, JP1.2, JP1.7, JP2.2, JP2.7, JP5.6, JP6.1, JP7.GND, Q10.S, Q11.S, Q9.S, R9.P$1; no longer C1.2, C12.-, C13.-, C16.2, JP1.1, JP2.6, JP5.2, JP5.7, JP6.2, JP6.7, Q1.S, Q2.S, Q3.S, R2.P$1
- net G_UART: now also JP1.6, JP2.6, JP5.3; no longer JP2.3, JP5.6, JP6.6
- net N$11: now also R2.P$2; no longer R10.P$2
- net N$12: now also Q1.D, R11.P$2; no longer J2.VDD
- net N$13: now also Q2.D, R12.P$2; no longer J2.VSS(GND)
- net N$14: now also Q3.D, R13.P$2; no longer J2.ICSP_DAT/PGD
- net N$15: now also Q12.D, R14.P$2; no longer J2.ICSP_CLK/PGC
- net N$9: now also JP6.2, R10.P$1; no longer JP1.2, R9.P$1
- net NRST: now also JP7.RST
- net RFET1: now also Q1.G, RN3D.2; no longer Q9.G, RN4D.2
- net RFET2: now also Q2.G, RN3C.2, SJ2.2; no longer Q10.G, RN4C.2, SJ1.2
- net RFET3: now also Q3.G, RN3B.2, SJ1.2; no longer Q11.G, RN4B.2, SJ2.2
- net RFET4: now also Q12.G, RN3A.2; no longer Q16.G, RN4A.2
- net RFET5: now also Q13.G, RN4D.2; no longer Q15.G, RN3D.2
- net RFET6: now also JP5.2, RN4A.2; no longer JP2.2, RN3A.2
- net RFET7: now also Q15.G, RN4B.2; no longer Q13.G, RN3B.2
- net RFET8: now also Q16.G, RN4C.2; no longer Q12.G, RN3C.2
- net ROW1: now also LED57.A, LED58.A, LED59.A, LED60.A, LED61.A, LED62.A, LED63.A, LED64.A, R11.P$1; no longer LED1.A, LED2.A, LED3.A, LED4.A, LED5.A, LED6.A, LED7.A, LED8.A, Q9.D
- net ROW2: now also LED49.A, LED50.A, LED51.A, LED52.A, LED53.A, LED54.A, LED55.A, LED56.A, R12.P$1; no longer LED10.A, LED11.A, LED12.A, LED13.A, LED14.A, LED15.A, LED16.A, LED9.A, Q10.D
- net ROW3: now also LED41.A, LED42.A, LED43.A, LED44.A, LED45.A, LED46.A, LED47.A, LED48.A, R13.P$1; no longer LED17.A, LED18.A, LED19.A, LED20.A, LED21.A, LED22.A, LED23.A, LED24.A, Q11.D
- net ROW4: now also LED33.A, LED34.A, LED35.A, LED36.A, LED37.A, LED38.A, LED39.A, LED40.A, R14.P$1; no longer LED25.A, LED26.A, LED27.A, LED28.A, LED29.A, LED30.A, LED31.A, LED32.A, Q16.D
- net ROW5: now also LED25.A, LED26.A, LED27.A, LED28.A, LED29.A, LED30.A, LED31.A, LED32.A, R15.P$1; no longer LED33.A, LED34.A, LED35.A, LED36.A, LED37.A, LED38.A, LED39.A, LED40.A, Q15.D
- net ROW6: now also LED17.A, LED18.A, LED19.A, LED20.A, LED21.A, LED22.A, LED23.A, LED24.A, R16.P$1; no longer LED41.A, LED42.A, LED43.A, LED44.A, LED45.A, LED46.A, LED47.A, LED48.A, Q14.D
- net ROW7: now also LED10.A, LED11.A, LED12.A, LED13.A, LED14.A, LED15.A, LED16.A, LED9.A, R17.P$1; no longer LED49.A, LED50.A, LED51.A, LED52.A, LED53.A, LED54.A, LED55.A, LED56.A, Q13.D
- net ROW8: now also LED1.A, LED2.A, LED3.A, LED4.A, LED5.A, LED6.A, LED7.A, LED8.A, R18.P$1; no longer LED57.A, LED58.A, LED59.A, LED60.A, LED61.A, LED62.A, LED63.A, LED64.A, Q12.D
- net SHIFT_LEFT: now also JP2.4; no longer JP4.4
- net SWCLK: now also JP7.SWCLK, SJ1.1; no longer SJ2.1
- net SWDAT: now also JP7.SWDAT, SJ2.1; no longer SJ1.1
Other:
- moved on the sheet: C10, C11, C14, C15, C2, C3, C4, C5, C6, C7, C8, C9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
