File: board_8x8_stm32/8x8_stm32.brd (EAGLE design)
At the start: 100 x 100 mm, 121 parts, among them IC1 STM32F0, J1 SWD_SHROUD, Q1 BSS123, Q10 BSS84, Q11 BSS84, Q12 BSS84, Q13 BSS84, Q14 BSS84, Q15 BSS84, Q16 BSS84, Q2 BSS123, Q3 BSS123, Q4 BSS123, Q5 BSS123, Q6 BSS123, Q7 BSS123, Q8 BSS123, Q9 BSS84

Commit message: almost done
Parts:
- added J2: (no value), tag-connect:TC2030-MCP-NL
- added T1: (no value), transistor-neu-to92:TO92
- added T2: (no value), transistor-neu-to92:TO92-BCE
- moved JP5 11.2 mm to (41.1, 13.0)
- moved JP4 10.8 mm to (13.0, 58.9)
- moved Q12 3.26 mm to (63.6, 12.2)
- moved Q13 1.68 mm to (61.2, 18.7)
- moved R10 1.15 mm to (52.0, 57.9)
- moved JP3 0.75 mm to (97.0, 58.9)
- moved R8 0.67 mm to (57.2, 59.4)
- moved C11 0.64 mm to (49.6, 57.4)
- moved RN4 0.50 mm to (74.5, 54.0)
- moved C5 0.35 mm to (44.0, 38.8)
- moved C7 0.35 mm to (50.5, 38.8)
- moved R5 0.35 mm to (42.5, 38.8)
- moved R7 0.35 mm to (49.0, 38.8)
- moved C8 0.28 mm to (54.2, 58.6)
- moved C6 0.25 mm to (45.8, 38.8)
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Connections:
- new net N$12: J2.2
- new net N$13: J2.3
- new net N$14: J2.4
- new net N$15: J2.5
Routing:
- net +5V: track 543.7 -> 197.6 mm, vias 10 -> 12
- net +3V3: track 477.8 -> 242.0 mm, vias 22 -> 23
- net G_UART: track 280.9 -> 263.3 mm
- net ROW4: track 153.3 -> 168.7 mm, vias 8 -> 10
- net GND: track 55.2 -> 69.0 mm
- net COMMS_LEFT: track 55.1 -> 43.4 mm
- net SHIFT_LEFT: track 69.3 -> 58.2 mm
- net COL8: track 177.9 -> 167.4 mm, vias 3 -> 4
- net COMMS_DOWN: track 77.3 -> 67.6 mm
- net ROW5: track 173.7 -> 182.5 mm, vias 9 -> 10
- net COL4: track 132.1 -> 137.7 mm, vias 9 -> 12
- net COL5: track 198.3 -> 193.6 mm, vias 8 -> 10
- net ROW3: track 149.7 -> 145.6 mm
- net RFET8: track 52.5 -> 48.9 mm
- net ROW7: track 138.2 -> 141.6 mm, vias 8 -> 6
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- added copper zone on layer 16, net +3V3
- added copper zone on layer 1, net +5V

Commit message: some prodding
Parts:
- flipped J1 to the top, turned to 270 degrees
Routing:
- net +3V3: track 242.0 -> 236.5 mm
- net NRST: track 49.8 -> 48.3 mm
- net SWCLK: track 47.1 -> 45.7 mm

Commit message: first prototype almost done
Parts:
- removed J2: (no value), tag-connect:TC2030-MCP-NL
- removed RN1, RN2: (no value), resistor-dil:EXB38V
- removed T1: (no value), transistor-neu-to92:TO92
- removed T2: (no value), transistor-neu-to92:TO92-BCE
- added JP7: TC2030-SWDNL, tag-connect:TC2030-MCP-NL
- added R11, R12, R13, R14, R15, R16, R17, R18: (no value), passives-7351:R0603-N
- C1: value 100p -> (none); device passives-7351:C0603-N -> rcl:E2-4
- C10, C9: value (none) -> 100p
- C12: device rcl:E2-4 -> passives-7351:C0603-N
- C13: value (none) -> 100p; device rcl:E2-4 -> passives-7351:C0603-N
- C14, C15: value (none) -> 100p; device rcl:C050-025X075 -> passives-7351:C0603-N
- C16: device passives-7351:C0603-N -> rcl:E2-4
- C2, C3: value 100p -> (none); device passives-7351:C0603-N -> rcl:C050-025X075
- C5, C6: value 100p -> (none)
- JP1: device Mine:1X02 -> SparkFun-Connectors:1X08_ROUND
- JP2: device SparkFun-Connectors:1X06 -> SparkFun-Connectors:1X08_ROUND
- JP5: device SparkFun-Connectors:1X08_ROUND -> SparkFun-Connectors:1X06
- JP6: device SparkFun-Connectors:1X08_ROUND -> Mine:1X02
- Q1, Q2, Q3: value BSS123 -> BSS84
- Q10, Q11, Q9: value BSS84 -> BSS123
- R10: value 2k2 -> (none)
- R2: value DNP -> 2k2
- R9: value (none) -> DNP
- moved LED1 123.7 mm to (93.8, 6.25)
- moved LED57 123.7 mm to (93.8, 93.8)
- moved LED64 123.7 mm to (6.25, 93.8)
- moved LED8 123.7 mm to (6.25, 6.25)
- moved LED16 107.5 mm to (6.25, 18.8)
- moved LED2 107.5 mm to (81.2, 6.25)
- moved LED49 107.5 mm to (93.8, 81.2)
- moved LED56 107.5 mm to (6.25, 81.2)
- moved LED58 107.5 mm to (81.2, 93.8)
- moved LED63 107.5 mm to (18.8, 93.8)
- moved LED7 107.5 mm to (18.8, 6.25)
- moved LED9 107.5 mm to (93.8, 18.8)
- moved LED17 95.2 mm to (93.8, 31.2)
- moved LED24 95.2 mm to (6.25, 31.2)
- moved LED3 95.2 mm to (68.8, 6.25)
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- renumbered U$1 to Q17
Connections:
- removed net N$1: Q8.3, RN2.1
- removed net N$2: Q7.3, RN2.2
- removed net N$3: Q6.3, RN2.3
- removed net N$4: Q5.3, RN2.4
- removed net N$5: Q4.3, RN1.1
- removed net N$6: Q3.3, RN1.2
- removed net N$7: Q2.3, RN1.3
- removed net N$8: Q1.3, RN1.4
- new net N$16: Q13.3, R15.2
- new net N$17: Q14.3, R16.2
- new net N$18: Q15.3, R17.2
- new net N$19: Q16.3, R18.2
- net +3V3: now also C12.1, C2.1, C5.1, C6.1, JP1.5, JP2.5, JP5.4, JP7.1, R10.2; no longer C10.1, C15.1, C16.1, C9.1, JP2.4, JP5.5, JP6.5, R9.2
- net +5V: now also C1.+, C16.+, C3.1, JP1.1, JP1.8, JP2.1, JP2.8, Q1.2, Q2.2, Q3.2; no longer C12.+, C13.+, C14.1, JP5.1, JP5.8, JP6.1, JP6.8, Q10.2, Q11.2, Q9.2
- net CFET1: now also Q11.1; no longer Q1.1
- net CFET2: now also Q10.1; no longer Q2.1
- net CFET3: now also Q9.1; no longer Q3.1
- net CFET4: now also Q8.1; no longer Q4.1
- net CFET5: now also Q7.1; no longer Q5.1
- net CFET7: now also Q5.1; no longer Q7.1
- net CFET8: now also Q4.1; no longer Q8.1
- net COL1: now also C14.1, LED16.K, LED16.K1, LED24.K, LED24.K1, LED32.K, LED32.K1, LED40.K, LED40.K1, LED48.K, LED48.K1, LED56.K, LED56.K1, LED64.K, LED64.K1, LED8.K, LED8.K1, Q4.3, R8.2; no longer C6.1, LED1.K, LED1.K1, LED17.K, LED17.K1, LED25.K, LED25.K1, LED33.K, LED33.K1, LED41.K, LED41.K1, LED49.K, LED49.K1, LED57.K, LED57.K1, LED9.K, LED9.K1, R6.2, RN2.8
- net COL2: now also C13.1, LED15.K, LED15.K1, LED23.K, LED23.K1, LED31.K, LED31.K1, LED39.K, LED39.K1, LED47.K, LED47.K1, LED55.K, LED55.K1, LED63.K, LED63.K1, LED7.K, LED7.K1, Q5.3, R7.2; no longer C5.1, LED10.K, LED10.K1, LED18.K, LED18.K1, LED2.K, LED2.K1, LED26.K, LED26.K1, LED34.K, LED34.K1, LED42.K, LED42.K1, LED50.K, LED50.K1, LED58.K, LED58.K1, R5.2, RN2.7
- net COL3: now also C7.1, LED14.K, LED14.K1, LED22.K, LED22.K1, LED30.K, LED30.K1, LED38.K, LED38.K1, LED46.K, LED46.K1, LED54.K, LED54.K1, LED6.K, LED6.K1, LED62.K, LED62.K1, Q6.3; no longer C3.1, LED11.K, LED11.K1, LED19.K, LED19.K1, LED27.K, LED27.K1, LED3.K, LED3.K1, LED35.K, LED35.K1, LED43.K, LED43.K1, LED51.K, LED51.K1, LED59.K, LED59.K1, RN2.6
- net COL4: now also C9.1, LED13.K, LED13.K1, LED21.K, LED21.K1, LED29.K, LED29.K1, LED37.K, LED37.K1, LED45.K, LED45.K1, LED5.K, LED5.K1, LED53.K, LED53.K1, LED61.K, LED61.K1, Q7.3, R6.2; no longer C4.1, LED12.K, LED12.K1, LED20.K, LED20.K1, LED28.K, LED28.K1, LED36.K, LED36.K1, LED4.K, LED4.K1, LED44.K, LED44.K1, LED52.K, LED52.K1, LED60.K, LED60.K1, R4.2, RN2.5
- net COL5: now also C15.1, LED12.K, LED12.K1, LED20.K, LED20.K1, LED28.K, LED28.K1, LED36.K, LED36.K1, LED4.K, LED4.K1, LED44.K, LED44.K1, LED52.K, LED52.K1, LED60.K, LED60.K1, Q8.3, R9.2; no longer C7.1, LED13.K, LED13.K1, LED21.K, LED21.K1, LED29.K, LED29.K1, LED37.K, LED37.K1, LED45.K, LED45.K1, LED5.K, LED5.K1, LED53.K, LED53.K1, LED61.K, LED61.K1, R7.2, RN1.8
- net COL6: now also C8.1, LED11.K, LED11.K1, LED19.K, LED19.K1, LED27.K, LED27.K1, LED3.K, LED3.K1, LED35.K, LED35.K1, LED43.K, LED43.K1, LED51.K, LED51.K1, LED59.K, LED59.K1, Q9.3, R4.2; no longer C2.1, LED14.K, LED14.K1, LED22.K, LED22.K1, LED30.K, LED30.K1, LED38.K, LED38.K1, LED46.K, LED46.K1, LED54.K, LED54.K1, LED6.K, LED6.K1, LED62.K, LED62.K1, R2.2, RN1.7
- net COL7: now also C10.1, LED10.K, LED10.K1, LED18.K, LED18.K1, LED2.K, LED2.K1, LED26.K, LED26.K1, LED34.K, LED34.K1, LED42.K, LED42.K1, LED50.K, LED50.K1, LED58.K, LED58.K1, Q10.3, R5.2; no longer C1.1, LED15.K, LED15.K1, LED23.K, LED23.K1, LED31.K, LED31.K1, LED39.K, LED39.K1, LED47.K, LED47.K1, LED55.K, LED55.K1, LED63.K, LED63.K1, LED7.K, LED7.K1, R1.2, RN1.6
- net COL8: now also C4.1, LED1.K, LED1.K1, LED17.K, LED17.K1, LED25.K, LED25.K1, LED33.K, LED33.K1, LED41.K, LED41.K1, LED49.K, LED49.K1, LED57.K, LED57.K1, LED9.K, LED9.K1, Q11.3, R1.2, R2.1; no longer C8.1, LED16.K, LED16.K1, LED24.K, LED24.K1, LED32.K, LED32.K1, LED40.K, LED40.K1, LED48.K, LED48.K1, LED56.K, LED56.K1, LED64.K, LED64.K1, LED8.K, LED8.K1, R10.1, R8.2, RN1.5
- net COMMS_DOWN: now also JP4.3; no longer JP5.3
- net COMMS_LEFT: now also JP2.3; no longer JP4.3
- net COMMS_UP: now also JP1.3; no longer JP6.3
- net GND: now also C1.-, C12.2, C13.2, C16.-, JP1.2, JP1.7, JP2.2, JP2.7, JP5.6, JP6.1, JP7.5, Q10.2, Q11.2, Q9.2, R9.1; no longer C1.2, C12.-, C13.-, C16.2, JP1.1, JP2.6, JP5.2, JP5.7, JP6.2, JP6.7, Q1.2, Q2.2, Q3.2, R2.1
- net G_UART: now also JP1.6, JP2.6, JP5.3; no longer JP2.3, JP5.6, JP6.6
- net N$11: now also R2.2; no longer R10.2
- net N$12: now also Q1.3, R11.2; no longer J2.2
- net N$13: now also Q2.3, R12.2; no longer J2.3
- net N$14: now also Q3.3, R13.2; no longer J2.4
- net N$15: now also Q12.3, R14.2; no longer J2.5
- net N$9: now also JP6.2, R10.1; no longer JP1.2, R9.1
- net NRST: now also JP7.3
- net RFET1: now also Q1.1, RN3.5; no longer Q9.1, RN4.5
- net RFET2: now also Q2.1, RN3.6, SJ2.2; no longer Q10.1, RN4.6, SJ1.2
- net RFET3: now also Q3.1, RN3.7, SJ1.2; no longer Q11.1, RN4.7, SJ2.2
- net RFET4: now also Q12.1, RN3.8; no longer Q16.1, RN4.8
- net RFET5: now also Q13.1, RN4.5; no longer Q15.1, RN3.5
- net RFET6: now also JP5.2, RN4.8; no longer JP2.2, RN3.8
- net RFET7: now also Q15.1, RN4.7; no longer Q13.1, RN3.7
- net RFET8: now also Q16.1, RN4.6; no longer Q12.1, RN3.6
- net ROW1: now also LED57.A, LED57.A1, LED58.A, LED58.A1, LED59.A, LED59.A1, LED60.A, LED60.A1, LED61.A, LED61.A1, LED62.A, LED62.A1, LED63.A, LED63.A1, LED64.A, LED64.A1, R11.1; no longer LED1.A, LED1.A1, LED2.A, LED2.A1, LED3.A, LED3.A1, LED4.A, LED4.A1, LED5.A, LED5.A1, LED6.A, LED6.A1, LED7.A, LED7.A1, LED8.A, LED8.A1, Q9.3
- net ROW2: now also LED49.A, LED49.A1, LED50.A, LED50.A1, LED51.A, LED51.A1, LED52.A, LED52.A1, LED53.A, LED53.A1, LED54.A, LED54.A1, LED55.A, LED55.A1, LED56.A, LED56.A1, R12.1; no longer LED10.A, LED10.A1, LED11.A, LED11.A1, LED12.A, LED12.A1, LED13.A, LED13.A1, LED14.A, LED14.A1, LED15.A, LED15.A1, LED16.A, LED16.A1, LED9.A, LED9.A1, Q10.3
- net ROW3: now also LED41.A, LED41.A1, LED42.A, LED42.A1, LED43.A, LED43.A1, LED44.A, LED44.A1, LED45.A, LED45.A1, LED46.A, LED46.A1, LED47.A, LED47.A1, LED48.A, LED48.A1, R13.1; no longer LED17.A, LED17.A1, LED18.A, LED18.A1, LED19.A, LED19.A1, LED20.A, LED20.A1, LED21.A, LED21.A1, LED22.A, LED22.A1, LED23.A, LED23.A1, LED24.A, LED24.A1, Q11.3
- net ROW4: now also LED33.A, LED33.A1, LED34.A, LED34.A1, LED35.A, LED35.A1, LED36.A, LED36.A1, LED37.A, LED37.A1, LED38.A, LED38.A1, LED39.A, LED39.A1, LED40.A, LED40.A1, R14.1; no longer LED25.A, LED25.A1, LED26.A, LED26.A1, LED27.A, LED27.A1, LED28.A, LED28.A1, LED29.A, LED29.A1, LED30.A, LED30.A1, LED31.A, LED31.A1, LED32.A, LED32.A1, Q16.3
- net ROW5: now also LED25.A, LED25.A1, LED26.A, LED26.A1, LED27.A, LED27.A1, LED28.A, LED28.A1, LED29.A, LED29.A1, LED30.A, LED30.A1, LED31.A, LED31.A1, LED32.A, LED32.A1, R15.1; no longer LED33.A, LED33.A1, LED34.A, LED34.A1, LED35.A, LED35.A1, LED36.A, LED36.A1, LED37.A, LED37.A1, LED38.A, LED38.A1, LED39.A, LED39.A1, LED40.A, LED40.A1, Q15.3
- net ROW6: now also LED17.A, LED17.A1, LED18.A, LED18.A1, LED19.A, LED19.A1, LED20.A, LED20.A1, LED21.A, LED21.A1, LED22.A, LED22.A1, LED23.A, LED23.A1, LED24.A, LED24.A1, R16.1; no longer LED41.A, LED41.A1, LED42.A, LED42.A1, LED43.A, LED43.A1, LED44.A, LED44.A1, LED45.A, LED45.A1, LED46.A, LED46.A1, LED47.A, LED47.A1, LED48.A, LED48.A1, Q14.3
- net ROW7: now also LED10.A, LED10.A1, LED11.A, LED11.A1, LED12.A, LED12.A1, LED13.A, LED13.A1, LED14.A, LED14.A1, LED15.A, LED15.A1, LED16.A, LED16.A1, LED9.A, LED9.A1, R17.1; no longer LED49.A, LED49.A1, LED50.A, LED50.A1, LED51.A, LED51.A1, LED52.A, LED52.A1, LED53.A, LED53.A1, LED54.A, LED54.A1, LED55.A, LED55.A1, LED56.A, LED56.A1, Q13.3
- net ROW8: now also LED1.A, LED1.A1, LED2.A, LED2.A1, LED3.A, LED3.A1, LED4.A, LED4.A1, LED5.A, LED5.A1, LED6.A, LED6.A1, LED7.A, LED7.A1, LED8.A, LED8.A1, R18.1; no longer LED57.A, LED57.A1, LED58.A, LED58.A1, LED59.A, LED59.A1, LED60.A, LED60.A1, LED61.A, LED61.A1, LED62.A, LED62.A1, LED63.A, LED63.A1, LED64.A, LED64.A1, Q12.3
- net SHIFT_LEFT: now also JP2.4; no longer JP4.4
- net SWCLK: now also JP7.4, SJ1.1; no longer SJ2.1
- net SWDAT: now also JP7.2, SJ2.1; no longer SJ1.1
Routing:
- net NRST: track 48.3 -> 69.9 mm, vias 6 -> 9
- net +3V3: track 236.5 -> 255.3 mm
- net SWCLK: track 45.7 -> 59.9 mm, vias 4 -> 5
- net SWDAT: track 53.3 -> 62.8 mm
- net COL8: track 167.4 -> 176.7 mm
- net N$8: track 8.29 -> 0.00 mm
- net N$4: track 7.54 -> 0.00 mm
- net N$7: track 5.86 -> 0.00 mm
- net COL7: track 160.1 -> 165.6 mm
- net GND: track 69.0 -> 74.2 mm, vias 28 -> 29
- net ROW8: track 170.8 -> 165.9 mm
- net N$19: track 0.00 -> 4.62 mm
- net +5V: track 197.6 -> 193.2 mm, vias 12 -> 14
- net COL5: track 193.6 -> 197.6 mm
- net N$1: track 3.82 -> 0.00 mm
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Other:
- board text added: "SWD"

Commit message: changed something...
Routing:
- net +5V: track 193.2 -> 199.2 mm, vias 14 -> 13
Changed lines of the file:
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@@
 <grid distance="0.25" unitdist="mm" unit="mm" style="lines" multiple="1" display="no" altdistance="0.125" altunitdist="mm" altunit="mm"/>
 <layers>
-<layer number="1" name="Top" color="4" fill="1" visible="no" active="yes"/>
-<layer number="16" name="Bottom" color="1" fill="1" visible="no" active="yes"/>
-<layer number="17" name="Pads" color="2" fill="1" visible="no" active="yes"/>
-<layer number="18" name="Vias" color="2" fill="1" visible="no" active="yes"/>
-<layer number="19" name="Unrouted" color="6" fill="1" visible="no" active="yes"/>
-<layer number="20" name="Dimension" color="15" fill="1" visible="no" active="yes"/>
-<layer number="21" name="tPlace" color="7" fill="1" visible="no" active="yes"/>
-<layer number="22" name="bPlace" color="7" fill="1" visible="no" active="yes"/>
-<layer number="23" name="tOrigins" color="15" fill="1" visible="no" active="yes"/>
+<layer number="1" name="Top" color="4" fill="1" visible="yes" active="yes"/>
+<layer number="16" name="Bottom" color="1" fill="1" visible="yes" active="yes"/>
+<layer number="17" name="Pads" color="2" fill="1" visible="yes" active="yes"/>
+<layer number="18" name="Vias" color="2" fill="1" visible="yes" active="yes"/>
+<layer number="19" name="Unrouted" color="6" fill="1" visible="yes" active="yes"/>
+<layer number="20" name="Dimension" color="15" fill="1" visible="yes" active="yes"/>
+<layer number="21" name="tPlace" color="7" fill="1" visible="yes" active="yes"/>
+<layer number="22" name="bPlace" color="7" fill="1" visible="yes" active="yes"/>
+<layer number="23" name="tOrigins" color="15" fill="1" visible="yes" active="yes"/>
 <layer number="24" name="bOrigins" color="15" fill="1" visible="no" active="yes"/>
 <layer number="25" name="tNames" color="7" fill="1" visible="no" active="yes"/>
@@
 <contactref element="RN4" pad="2"/>
 <contactref element="RN4" pad="3"/>
-<wire x1="78.52" y1="76.32" x2="78.52" y2="74" width="0.6096" layer="1"/>
-<wire x1="78.52" y1="74" x2="78.52" y2="72.48" width="0.6096" layer="1"/>
-<wire x1="78.52" y1="72.48" x2="79" y2="72" width="0.6096" layer="1"/>
-<wire x1="79" y1="72" x2="79" y2="71.75" width="0.6096" layer="1"/>
+<wire x1="78.52" y1="74" x2="78.52" y2="72.23" width="0.6096" layer="1"/>
 <via x="79" y="71.75" extent="1-16" drill="0.381" shape="octagon"/>
 <wire x1="79" y1="71.75" x2="78.75" y2="71.5" width="0.6096" layer="16"/>
@@
 <wire x1="78.75" y1="81.75" x2="78.75" y2="80.5" width="0.6096" layer="1"/>
 <wire x1="78.75" y1="80.5" x2="79" y2="80.25" width="0.6096" layer="1"/>
-<wire x1="79" y1="80.25" x2="79" y2="77.55" width="0.6096" layer="1"/>
-<wire x1="79" y1="77.55" x2="78.52" y2="76.32" width="0.6096" layer="1"/>
+<wire x1="79" y1="80.25" x2="79" y2="76.8" width="0.6096" layer="1"/>
 <wire x1="63.625" y1="33.1" x2="63.625" y2="33.975" width="0.254" layer="1"/>
 <wire x1="63.625" y1="34.775" x2="63.625" y2="35.65" width="0.254" layer="1"/>
@@
 <wire x1="79" y1="52" x2="79" y2="50.76" width="0.6096" layer="1"/>
 <wire x1="79" y1="50.76" x2="78.93" y2="50.69" width="0.6096" layer="1"/>
-<wire x1="73.75" y1="73.984" x2="78.504" y2="73.984" width="0.6096" layer="1"/>
 <wire x1="78.504" y1="73.984" x2="78.52" y2="74" width="0.6096" layer="1"/>
-<via x="80.765" y="91.39" extent="1-16" drill="0.381" shape="octagon"/>
-<wire x1="83.75" y1="92.75" x2="83.75" y2="96.375" width="0.6096" layer="16"/>
-<via x="83.75" y="96.375" extent="1-16" drill="0.381" shape="octagon"/>
 <wire x1="62.016" y1="24.25" x2="64.5" y2="24.25" width="0.6096" layer="1"/>
 <wire x1="64.5" y1="24.25" x2="65.25" y2="23.5" width="0.6096" layer="1"/>
@@
 <wire x1="12.595" y1="41.095" x2="12" y2="40.5" width="2.1844" layer="1"/>
 <wire x1="12" y1="40.5" x2="2.25" y2="40.5" width="2.1844" layer="1"/>
-<wire x1="83.75" y1="92.75" x2="82.75" y2="91.75" width="0.6096" layer="16"/>
-<wire x1="82.75" y1="91.75" x2="81.125" y2="91.75" width="0.6096" layer="16"/>
-<wire x1="81.125" y1="91.75" x2="80.765" y2="91.39" width="0.6096" layer="16"/>
-<wire x1="80.765" y1="91.39" x2="80.765" y2="89.275" width="0.6096" layer="1"/>
-<wire x1="80.765" y1="89.275" x2="80.39" y2="88.9" width="0.6096" layer="1"/>
 <wire x1="79" y1="86.75" x2="80.5" y2="88.25" width="0.6096" layer="1"/>
 <wire x1="80.5" y1="88.25" x2="80.5" y2="88.79" width="0.6096" layer="1"/>
 <wire x1="80.5" y1="88.79" x2="80.39" y2="88.9" width="0.6096" layer="1"/>
 <wire x1="2.375" y1="59" x2="14" y2="58.875" width="2.1844" layer="1"/>
-<via x="83.75" y="94.875" extent="1-16" drill="0.381" shape="octagon"/>
-<via x="83.75" y="95.625" extent="1-16" drill="0.381" shape="octagon"/>
 <wire x1="65.5" y1="6" x2="65.5" y2="7" width="0.6096" layer="1"/>
 <wire x1="65.5" y1="7" x2="66" y2="7.5" width="0.6096" layer="1"/>
@@
 <wire x1="63.625" y1="35.65" x2="63.625" y2="37.265" width="0.254" layer="1"/>
 <wire x1="63.625" y1="37.265" x2="63.8" y2="37.44" width="0.254" layer="1"/>
+<wire x1="79" y1="71.75" x2="79" y2="72" width="0.6096" layer="16"/>
+<wire x1="79" y1="72" x2="80.25" y2="72" width="0.6096" layer="16"/>
+<wire x1="80.25" y1="72" x2="81" y2="71.25" width="0.6096" layer="16"/>
+<wire x1="81" y1="71.25" x2="81" y2="71" width="0.6096" layer="16"/>
+<via x="81" y="71" extent="1-16" drill="0.381" shape="octagon"/>
+<wire x1="81" y1="71" x2="91.25" y2="71" width="0.6096" layer="1"/>
+<wire x1="91.25" y1="71" x2="91.5" y2="71.25" width="0.6096" layer="1"/>
+<via x="91.5" y="71.25" extent="1-16" drill="0.381" shape="octagon"/>
+<wire x1="91.5" y1="71.25" x2="93.5" y2="71.25" width="0.6096" layer="16"/>
+<via x="93.5" y="71.25" extent="1-16" drill="0.381" shape="octagon"/>
+<wire x1="93.5" y1="71.25" x2="93.5" y2="71.5" width="0.6096" layer="1"/>
+<wire x1="78.52" y1="72.23" x2="79" y2="71.75" width="0.6096" layer="1"/>
+<wire x1="79" y1="76.8" x2="78.52" y2="76.32" width="0.6096" layer="1"/>
+<wire x1="73.75" y1="73.984" x2="74.734" y2="73.984" width="0.6096" layer="1"/>
+<wire x1="74.734" y1="73.984" x2="74.75" y2="74" width="0.6096" layer="1"/>
+<wire x1="74.75" y1="74" x2="78.25" y2="74" width="1.016" layer="1"/>
+<wire x1="78.25" y1="74" x2="78.488" y2="74" width="1.016" layer="1"/>
+<wire x1="78.488" y1="74" x2="78.504" y2="73.984" width="1.016" layer="1"/>
+<wire x1="78.52" y1="76.32" x2="78.52" y2="74.27" width="1.016" layer="1"/>
+<wire x1="78.52" y1="74.27" x2="78.25" y2="74" width="1.016" layer="1"/>
 </signal>
 <signal name="N$9">
